File: projects/DAC_R.sch (KiCad schematic (older format))
At the start: 13 parts, among them U301 WM874XX

Commit message: updated LED indicators in schematic files (*.sch)
Parts:
- added D?: RED_LED, symbol RED_LED
- added R?: R, symbol R
Connections:
- no-connect marks 2 -> 1
Changed lines of the file:
@@
 LIBS:microchip_gosselin
 LIBS:linear_technology_gosselin
+LIBS:led_gosselin
 LIBS:mStereo2-cache
 EELAYER 24 0
@@
 Wire Wire Line
 	6700 2800 6700 3800
-NoConn ~ 6500 4000
 Wire Wire Line
 	4350 4450 4350 4300
@@
 Connection ~ 4900 2800
 NoConn ~ 6500 3900
+$Comp
+L RED_LED D?
+U 1 1 5455D948
+P 6900 4000
+F 0 "D?" H 6900 4100 50  0000 C CNN
+F 1 "RED_LED" H 6900 3900 50  0000 C CNN
+F 2 "" H 6900 4000 60  0000 C CNN
+F 3 "" H 6900 4000 60  0000 C CNN
+F 4 "160-1427-1-ND" H 7100 4300 60  0001 C CNN "Supplier-PN"
+F 5 "Digi-key" H 7000 4200 60  0001 C CNN "Supplier"
+F 6 "LED SUPER RED CLR THIN 0805 SMD" H 7400 4600 60  0001 C CNN "Description"
+F 7 "Lite-On" H 7200 4400 60  0001 C CNN "Manu"
+F 8 "LTST-C171KRKT" H 7300 4500 60  0001 C CNN "Manu-PN"
+	1    6900 4000
+	1    0    0    -1
+$EndComp
+$Comp
+L R R?
+U 1 1 5455D997
+P 7700 4000
+F 0 "R?" V 7780 4000 40  0000 C CNN
+F 1 "R" V 7707 4001 40  0000 C CNN
+F 2 "" V 7630 4000 30  0000 C CNN
+F 3 "" H 7700 4000 30  0000 C CNN
+F 4 "Digi-Key" H 7700 4000 60  0001 C CNN "Supplier"
+F 5 "RNCP0805FTD121RCT-ND" H 7700 4000 60  0001 C CNN "Supplier-PN"
+F 6 "Stackpole" H 7700 4000 60  0001 C CNN "Manu"
+F 7 "RNCP0805FTD121R" H 7700 4000 60  0001 C CNN "Manu-PN"
+F 8 "RES 121 OHM 1/4W 1% 0805" H 7700 4000 60  0001 C CNN "Description"
+	1    7700 4000
+	0    -1   -1   0
+$EndComp
 $EndSCHEMATC

Commit message: updated LEDs in schematic, output connectors, re-annotated
Parts:
- R301: renamed from R?; value R -> 121
- gave numbers to parts that had none: 1
Connections:
- wire segments 57 -> 61
Other:
- moved on the sheet: R301
Changed lines of the file:
@@
 Connection ~ 3600 4100
 Wire Wire Line
-	2750 5100 8800 5100
+	2750 5100 9050 5100
 Wire Wire Line
 	8800 5100 8800 4850
@@
 NoConn ~ 6500 3900
 $Comp
-L RED_LED D?
+L RED_LED D301
 U 1 1 5455D948
 P 6900 4000
-F 0 "D?" H 6900 4100 50  0000 C CNN
+F 0 "D301" H 6900 4100 50  0000 C CNN
 F 1 "RED_LED" H 6900 3900 50  0000 C CNN
 F 2 "" H 6900 4000 60  0000 C CNN
@@
 $EndComp
 $Comp
-L R R?
+L R R301
 U 1 1 5455D997
-P 7700 4000
-F 0 "R?" V 7780 4000 40  0000 C CNN
-F 1 "R" V 7707 4001 40  0000 C CNN
-F 2 "" V 7630 4000 30  0000 C CNN
-F 3 "" H 7700 4000 30  0000 C CNN
-F 4 "Digi-Key" H 7700 4000 60  0001 C CNN "Supplier"
-F 5 "RNCP0805FTD121RCT-ND" H 7700 4000 60  0001 C CNN "Supplier-PN"
-F 6 "Stackpole" H 7700 4000 60  0001 C CNN "Manu"
-F 7 "RNCP0805FTD121R" H 7700 4000 60  0001 C CNN "Manu-PN"
-F 8 "RES 121 OHM 1/4W 1% 0805" H 7700 4000 60  0001 C CNN "Description"
-	1    7700 4000
+P 7450 4000
+F 0 "R301" V 7530 4000 40  0000 C CNN
+F 1 "121" V 7457 4001 40  0000 C CNN
+F 2 "" V 7380 4000 30  0000 C CNN
+F 3 "" H 7450 4000 30  0000 C CNN
+F 4 "Digi-Key" H 7450 4000 60  0001 C CNN "Supplier"
+F 5 "RNCP0805FTD121RCT-ND" H 7450 4000 60  0001 C CNN "Supplier-PN"
+F 6 "Stackpole" H 7450 4000 60  0001 C CNN "Manu"
+F 7 "RNCP0805FTD121R" H 7450 4000 60  0001 C CNN "Manu-PN"
+F 8 "RES 121 OHM 1/4W 1% 0805" H 7450 4000 60  0001 C CNN "Description"
+	1    7450 4000
 	0    -1   -1   0
 $EndComp
+Wire Wire Line
+	6500 4000 6700 4000
+Wire Wire Line
+	7100 4000 7200 4000
+Wire Wire Line
+	7700 4000 9050 4000
+Wire Wire Line
+	9050 4000 9050 5100
+Connection ~ 8800 5100
 $EndSCHEMATC
