File: projects/DAC_R.sch (KiCad schematic (older format))
At the start: 15 parts, among them U301 WM874XX

Commit message: add box cap and small electrolytic cap footprints
Parts:
- removed C302, C304, C306, C308, C310, C312: 22, symbol C
- added c301, c302, c303, c304, c305, c306: 22, symbol CP1
- renumbered C303 to C302, C305 to C303, C307 to C304, C309 to C305, C311 to C306
Changed lines of the file:
@@
 DVDD
 $Comp
-L C C303
+L C C302
 U 1 1 544B8572
 P 3600 4650
-F 0 "C303" H 3600 4750 40  0000 L CNN
+F 0 "C302" H 3600 4750 40  0000 L CNN
 F 1 "0.1" H 3606 4565 40  0000 L CNN
 F 2 "" H 3638 4500 30  0000 C CNN
@@
 $EndComp
 $Comp
-L C C307
+L C C304
 U 1 1 544B8573
 P 7550 4650
-F 0 "C307" H 7550 4750 40  0000 L CNN
+F 0 "C304" H 7550 4750 40  0000 L CNN
 F 1 "0.1" H 7556 4565 40  0000 L CNN
 F 2 "" H 7588 4500 30  0000 C CNN
@@
 	6500 4100 8800 4100
 $Comp
-L C C305
+L C C303
 U 1 1 54153DC6
 P 4100 4650
-F 0 "C305" H 4100 4750 40  0000 L CNN
+F 0 "C303" H 4100 4750 40  0000 L CNN
 F 1 "0.1" H 4106 4565 40  0000 L CNN
 F 2 "" H 4138 4500 30  0000 C CNN
@@
 Connection ~ 4100 5100
 $Comp
-L C C309
+L C C305
 U 1 1 544B8575
 P 8050 4650
-F 0 "C309" H 8050 4750 40  0000 L CNN
+F 0 "C305" H 8050 4750 40  0000 L CNN
 F 1 "0.1" H 8056 4565 40  0000 L CNN
 F 2 "" H 8088 4500 30  0000 C CNN
@@
 	2750 2800 6700 2800
 $Comp
-L C C311
+L C C306
 U 1 1 544B8576
 P 8550 4650
-F 0 "C311" H 8550 4750 40  0000 L CNN
+F 0 "C306" H 8550 4750 40  0000 L CNN
 F 1 "0.1" H 8556 4565 40  0000 L CNN
 F 2 "" H 8588 4500 30  0000 C CNN
@@
 F 8 "CAP CER 0.1UF 16V 10% X7R 0805" H 8550 4650 60  0001 C CNN "Description"
 	1    8550 4650
-	1    0    0    -1
-$EndComp
-$Comp
-L C C302
-U 1 1 544B8577
-P 3350 4650
-F 0 "C302" H 3350 4750 40  0000 L CNN
-F 1 "22" H 3356 4565 40  0000 L CNN
-F 2 "" H 3388 4500 30  0000 C CNN
-F 3 "" H 3350 4650 60  0000 C CNN
-F 4 "Digi-Key" H 3350 4650 60  0001 C CNN "Supplier"
-F 5 "P16405CT-ND" H 3350 4650 60  0001 C CNN "Supplier-PN"
-F 6 "Panasonic" H 3350 4650 60  0001 C CNN "Manu"
-F 7 "32SEPF22M+TSS" H 3350 4650 60  0001 C CNN "Manu-PN"
-F 8 "CAP ALUM 22UF 32V 20% RADIAL" H 3350 4650 60  0001 C CNN "Description"
-	1    3350 4650
 	1    0    0    -1
 $EndComp
@@
 Connection ~ 7300 2650
 Connection ~ 7300 4450
-$Comp
-L C C304
-U 1 1 544A0699
-P 3850 4650
-F 0 "C304" H 3850 4750 40  0000 L CNN
-F 1 "22" H 3856 4565 40  0000 L CNN
-F 2 "" H 3888 4500 30  0000 C CNN
-F 3 "" H 3850 4650 60  0000 C CNN
-F 4 "Digi-Key" H 3850 4650 60  0001 C CNN "Supplier"
-F 5 "P16405CT-ND" H 3850 4650 60  0001 C CNN "Supplier-PN"
-F 6 "Panasonic" H 3850 4650 60  0001 C CNN "Manu"
-F 7 "32SEPF22M+TSS" H 3850 4650 60  0001 C CNN "Manu-PN"
-F 8 "CAP ALUM 22UF 32V 20% RADIAL" H 3850 4650 60  0001 C CNN "Description"
-	1    3850 4650
-	1    0    0    -1
-$EndComp
-$Comp
-L C C306
-U 1 1 544A06AE
-P 4350 4650
-F 0 "C306" H 4350 4750 40  0000 L CNN
-F 1 "22" H 4356 4565 40  0000 L CNN
-F 2 "" H 4388 4500 30  0000 C CNN
-F 3 "" H 4350 4650 60  0000 C CNN
-F 4 "Digi-Key" H 4350 4650 60  0001 C CNN "Supplier"
-F 5 "P16405CT-ND" H 4350 4650 60  0001 C CNN "Supplier-PN"
-F 6 "Panasonic" H 4350 4650 60  0001 C CNN "Manu"
-F 7 "32SEPF22M+TSS" H 4350 4650 60  0001 C CNN "Manu-PN"
-F 8 "CAP ALUM 22UF 32V 20% RADIAL" H 4350 4650 60  0001 C CNN "Description"
-	1    4350 4650
-	1    0    0    -1
-$EndComp
-$Comp
-L C C308
-U 1 1 544A076D
-P 7800 4650
-F 0 "C308" H 7800 4750 40  0000 L CNN
-F 1 "22" H 7806 4565 40  0000 L CNN
-F 2 "" H 7838 4500 30  0000 C CNN
-F 3 "" H 7800 4650 60  0000 C CNN
-F 4 "Digi-Key" H 7800 4650 60  0001 C CNN "Supplier"
-F 5 "P16405CT-ND" H 7800 4650 60  0001 C CNN "Supplier-PN"
-F 6 "Panasonic" H 7800 4650 60  0001 C CNN "Manu"
-F 7 "32SEPF22M+TSS" H 7800 4650 60  0001 C CNN "Manu-PN"
-F 8 "CAP ALUM 22UF 32V 20% RADIAL" H 7800 4650 60  0001 C CNN "Description"
-	1    7800 4650
-	1    0    0    -1
-$EndComp
-$Comp
-L C C310
-U 1 1 544A0796
-P 8300 4650
-F 0 "C310" H 8300 4750 40  0000 L CNN
-F 1 "22" H 8306 4565 40  0000 L CNN
-F 2 "" H 8338 4500 30  0000 C CNN
-F 3 "" H 8300 4650 60  0000 C CNN
-F 4 "Digi-Key" H 8300 4650 60  0001 C CNN "Supplier"
-F 5 "P16405CT-ND" H 8300 4650 60  0001 C CNN "Supplier-PN"
-F 6 "Panasonic" H 8300 4650 60  0001 C CNN "Manu"
-F 7 "32SEPF22M+TSS" H 8300 4650 60  0001 C CNN "Manu-PN"
-F 8 "CAP ALUM 22UF 32V 20% RADIAL" H 8300 4650 60  0001 C CNN "Description"
-	1    8300 4650
-	1    0    0    -1
-$EndComp
-$Comp
-L C C312
-U 1 1 544A07AB
-P 8800 4650
-F 0 "C312" H 8800 4750 40  0000 L CNN
-F 1 "22" H 8806 4565 40  0000 L CNN
-F 2 "" H 8838 4500 30  0000 C CNN
-F 3 "" H 8800 4650 60  0000 C CNN
-F 4 "Digi-Key" H 8800 4650 60  0001 C CNN "Supplier"
-F 5 "P16405CT-ND" H 8800 4650 60  0001 C CNN "Supplier-PN"
-F 6 "Panasonic" H 8800 4650 60  0001 C CNN "Manu"
-F 7 "32SEPF22M+TSS" H 8800 4650 60  0001 C CNN "Manu-PN"
-F 8 "CAP ALUM 22UF 32V 20% RADIAL" H 8800 4650 60  0001 C CNN "Description"
-	1    8800 4650
-	1    0    0    -1
-$EndComp
 Wire Wire Line
 	6500 3700 6700 3700
@@
 	9050 4000 9050 5100
 Connection ~ 8800 5100
+$Comp
+L CP1 c301
+U 1 1 548583ED
+P 3350 4650
+F 0 "c301" H 3400 4750 50  0000 L CNN
+F 1 "22" H 3400 4550 50  0000 L CNN
+F 2 "" H 3350 4650 60  0000 C CNN
+F 3 "" H 3350 4650 60  0000 C CNN
+F 4 "Digi-key" H 3350 4650 60  0001 C CNN "Supplier"
+F 5 "P16405CT-ND" H 3350 4650 60  0001 C CNN "Supplier-PN"
+F 6 "Panasonic" H 3350 4650 60  0001 C CNN "Manu"
+F 7 "32SEPF22M+TSS" H 3350 4650 60  0001 C CNN "Manu-PN"
+F 8 "CAP ALUM 22UF 32V 20% RADIAL" H 3350 4650 60  0001 C CNN "Description"
+	1    3350 4650
+	1    0    0    -1
+$EndComp
+$Comp
+L CP1 c302
+U 1 1 548584EC
+P 3850 4650
+F 0 "c302" H 3900 4750 50  0000 L CNN
+F 1 "22" H 3900 4550 50  0000 L CNN
+F 2 "" H 3850 4650 60  0000 C CNN
+F 3 "" H 3850 4650 60  0000 C CNN
+F 4 "Digi-key" H 3850 4650 60  0001 C CNN "Supplier"
+F 5 "P16405CT-ND" H 3850 4650 60  0001 C CNN "Supplier-PN"
+F 6 "Panasonic" H 3850 4650 60  0001 C CNN "Manu"
+F 7 "32SEPF22M+TSS" H 3850 4650 60  0001 C CNN "Manu-PN"
+F 8 "CAP ALUM 22UF 32V 20% RADIAL" H 3850 4650 60  0001 C CNN "Description"
+	1    3850 4650
+	1    0    0    -1
+$EndComp
+$Comp
+L CP1 c303
+U 1 1 54858501
+P 4350 4650
+F 0 "c303" H 4400 4750 50  0000 L CNN
+F 1 "22" H 4400 4550 50  0000 L CNN
+F 2 "" H 4350 4650 60  0000 C CNN
+F 3 "" H 4350 4650 60  0000 C CNN
+F 4 "Digi-key" H 4350 4650 60  0001 C CNN "Supplier"
+F 5 "P16405CT-ND" H 4350 4650 60  0001 C CNN "Supplier-PN"
+F 6 "Panasonic" H 4350 4650 60  0001 C CNN "Manu"
+F 7 "32SEPF22M+TSS" H 4350 4650 60  0001 C CNN "Manu-PN"
+F 8 "CAP ALUM 22UF 32V 20% RADIAL" H 4350 4650 60  0001 C CNN "Description"
+	1    4350 4650
+	1    0    0    -1
+$EndComp
+$Comp
+L CP1 c304
+U 1 1 54858516
+P 7800 4650
+F 0 "c304" H 7850 4750 50  0000 L CNN
+F 1 "22" H 7850 4550 50  0000 L CNN
+F 2 "" H 7800 4650 60  0000 C CNN
+F 3 "" H 7800 4650 60  0000 C CNN
+F 4 "Digi-key" H 7800 4650 60  0001 C CNN "Supplier"
+F 5 "P16405CT-ND" H 7800 4650 60  0001 C CNN "Supplier-PN"
+F 6 "Panasonic" H 7800 4650 60  0001 C CNN "Manu"
+F 7 "32SEPF22M+TSS" H 7800 4650 60  0001 C CNN "Manu-PN"
+F 8 "CAP ALUM 22UF 32V 20% RADIAL" H 7800 4650 60  0001 C CNN "Description"
+	1    7800 4650
+	1    0    0    -1
+$EndComp
+$Comp
+L CP1 c305
+U 1 1 5485853F
+P 8300 4650
+F 0 "c305" H 8350 4750 50  0000 L CNN
+F 1 "22" H 8350 4550 50  0000 L CNN
+F 2 "" H 8300 4650 60  0000 C CNN
+F 3 "" H 8300 4650 60  0000 C CNN
+F 4 "Digi-key" H 8300 4650 60  0001 C CNN "Supplier"
+F 5 "P16405CT-ND" H 8300 4650 60  0001 C CNN "Supplier-PN"
+F 6 "Panasonic" H 8300 4650 60  0001 C CNN "Manu"
+F 7 "32SEPF22M+TSS" H 8300 4650 60  0001 C CNN "Manu-PN"
+F 8 "CAP ALUM 22UF 32V 20% RADIAL" H 8300 4650 60  0001 C CNN "Description"
+	1    8300 4650
+	1    0    0    -1
+$EndComp
+$Comp
+L CP1 c306
+U 1 1 54858554
+P 8800 4650
+F 0 "c306" H 8850 4750 50  0000 L CNN
+F 1 "22" H 8850 4550 50  0000 L CNN
+F 2 "" H 8800 4650 60  0000 C CNN
+F 3 "" H 8800 4650 60  0000 C CNN
+F 4 "Digi-key" H 8800 4650 60  0001 C CNN "Supplier"
+F 5 "P16405CT-ND" H 8800 4650 60  0001 C CNN "Supplier-PN"
+F 6 "Panasonic" H 8800 4650 60  0001 C CNN "Manu"
+F 7 "32SEPF22M+TSS" H 8800 4650 60  0001 C CNN "Manu-PN"
+F 8 "CAP ALUM 22UF 32V 20% RADIAL" H 8800 4650 60  0001 C CNN "Description"
+	1    8800 4650
+	1    0    0    -1
+$EndComp
 $EndSCHEMATC

Commit message: update bom
Parts:
- U301: value WM874XX -> WM8741
Changed lines of the file:
@@
 P 5800 3950
 F 0 "U301" H 5800 3950 60  0000 C CNN
-F 1 "WM874XX" H 5850 4750 60  0000 C CNN
+F 1 "WM8741" H 5850 4750 60  0000 C CNN
 F 2 "" H 5800 3750 60  0000 C CNN
 F 3 "" H 5800 3750 60  0000 C CNN

Commit message: re-add netlist, correct part numbers
Parts:
- removed U301: WM8741, symbol WM874XX
- added U301: WM8741, symbol WM8741
- renumbered c301 to C302, C302 to C303, c302 to C304, C303 to C305, c303 to C306, C304 to C307, c304 to C308, C305 to C309, c305 to C310, C306 to C311, c306 to C312
Changed lines of the file:
@@
 LIBS:ti_gosselin
 LIBS:oscillator_gosselin
-LIBS:wolfson_gosselin
 LIBS:power
 LIBS:device
@@
 LIBS:linear_technology_gosselin
 LIBS:led_gosselin
-LIBS:mStereo2-cache
+LIBS:wolfson_gosselin
 EELAYER 24 0
 EELAYER END
@@
 Comment4 ""
 $EndDescr
-$Comp
-L WM874XX U301
-U 1 1 544B8571
-P 5800 3950
-F 0 "U301" H 5800 3950 60  0000 C CNN
-F 1 "WM8741" H 5850 4750 60  0000 C CNN
-F 2 "" H 5800 3750 60  0000 C CNN
-F 3 "" H 5800 3750 60  0000 C CNN
-F 4 "Mouser" H 5950 5000 60  0001 C CNN "Supplier"
-F 5 "238-WM8741GEDS/V" H 6300 5100 60  0001 C CNN "Supplier-PN"
-F 6 "Wolfson Microelectronics" H 6350 5200 60  0001 C CNN "Manu"
-F 7 "WM8741GEDS/V" H 6150 5300 60  0001 C CNN "Manu-PN"
-F 8 "Audio D/A Converter ICs Stereo DAC, High End " H 6900 5400 60  0001 C CNN "Description"
-	1    5800 3950
-	1    0    0    -1
-$EndComp
 Text HLabel 4750 3300 0    60   Input ~ 0
 LRCLK
@@
 DVDD
 $Comp
-L C C302
+L C C303
 U 1 1 544B8572
 P 3600 4650
-F 0 "C302" H 3600 4750 40  0000 L CNN
+F 0 "C303" H 3600 4750 40  0000 L CNN
 F 1 "0.1" H 3606 4565 40  0000 L CNN
 F 2 "" H 3638 4500 30  0000 C CNN
@@
 $EndComp
 $Comp
-L C C304
+L C C307
 U 1 1 544B8573
 P 7550 4650
-F 0 "C304" H 7550 4750 40  0000 L CNN
+F 0 "C307" H 7550 4750 40  0000 L CNN
 F 1 "0.1" H 7556 4565 40  0000 L CNN
 F 2 "" H 7588 4500 30  0000 C CNN
@@
 	6500 4100 8800 4100
 $Comp
-L C C303
+L C C305
 U 1 1 54153DC6
 P 4100 4650
-F 0 "C303" H 4100 4750 40  0000 L CNN
+F 0 "C305" H 4100 4750 40  0000 L CNN
 F 1 "0.1" H 4106 4565 40  0000 L CNN
 F 2 "" H 4138 4500 30  0000 C CNN
@@
 Connection ~ 4100 5100
 $Comp
-L C C305
+L C C309
 U 1 1 544B8575
 P 8050 4650
-F 0 "C305" H 8050 4750 40  0000 L CNN
+F 0 "C309" H 8050 4750 40  0000 L CNN
 F 1 "0.1" H 8056 4565 40  0000 L CNN
 F 2 "" H 8088 4500 30  0000 C CNN
@@
 	2750 2800 6700 2800
 $Comp
-L C C306
+L C C311
 U 1 1 544B8576
 P 8550 4650
-F 0 "C306" H 8550 4750 40  0000 L CNN
+F 0 "C311" H 8550 4750 40  0000 L CNN
 F 1 "0.1" H 8556 4565 40  0000 L CNN
 F 2 "" H 8588 4500 30  0000 C CNN
@@
 Connection ~ 8800 5100
 $Comp
-L CP1 c301
+L CP1 C302
 U 1 1 548583ED
 P 3350 4650
-F 0 "c301" H 3400 4750 50  0000 L CNN
+F 0 "C302" H 3400 4750 50  0000 L CNN
 F 1 "22" H 3400 4550 50  0000 L CNN
 F 2 "" H 3350 4650 60  0000 C CNN
@@
 $EndComp
 $Comp
-L CP1 c302
+L CP1 C304
 U 1 1 548584EC
 P 3850 4650
-F 0 "c302" H 3900 4750 50  0000 L CNN
+F 0 "C304" H 3900 4750 50  0000 L CNN
 F 1 "22" H 3900 4550 50  0000 L CNN
 F 2 "" H 3850 4650 60  0000 C CNN
@@
 $EndComp
 $Comp
-L CP1 c303
+L CP1 C306
 U 1 1 54858501
 P 4350 4650
-F 0 "c303" H 4400 4750 50  0000 L CNN
+F 0 "C306" H 4400 4750 50  0000 L CNN
 F 1 "22" H 4400 4550 50  0000 L CNN
 F 2 "" H 4350 4650 60  0000 C CNN
@@
 $EndComp
 $Comp
-L CP1 c304
+L CP1 C308
 U 1 1 54858516
 P 7800 4650
-F 0 "c304" H 7850 4750 50  0000 L CNN
+F 0 "C308" H 7850 4750 50  0000 L CNN
 F 1 "22" H 7850 4550 50  0000 L CNN
 F 2 "" H 7800 4650 60  0000 C CNN
@@
 $EndComp
 $Comp
-L CP1 c305
+L CP1 C310
 U 1 1 5485853F
 P 8300 4650
-F 0 "c305" H 8350 4750 50  0000 L CNN
+F 0 "C310" H 8350 4750 50  0000 L CNN
 F 1 "22" H 8350 4550 50  0000 L CNN
 F 2 "" H 8300 4650 60  0000 C CNN
@@
 $EndComp
 $Comp
-L CP1 c306
+L CP1 C312
 U 1 1 54858554
 P 8800 4650
-F 0 "c306" H 8850 4750 50  0000 L CNN
+F 0 "C312" H 8850 4750 50  0000 L CNN
 F 1 "22" H 8850 4550 50  0000 L CNN
 F 2 "" H 8800 4650 60  0000 C CNN
@@
 	1    0    0    -1
 $EndComp
+$Comp
+L WM8741 U301
+U 1 1 54D07BF0
+P 5800 3950
+F 0 "U301" H 5800 3950 60  0000 C CNN
+F 1 "WM8741" H 5850 4750 60  0000 C CNN
+F 2 "" H 5800 3750 60  0000 C CNN
+F 3 "" H 5800 3750 60  0000 C CNN
+F 4 "238-WM8741GEDS/V" H 6300 5100 60  0001 C CNN "Supplier-PN"
+F 5 "Mouser" H 5950 5000 60  0001 C CNN "Supplier"
+F 6 "Audio D/A Converter ICs Stereo DAC, High End " H 6900 5400 60  0001 C CNN "Description"
+F 7 "WM8741GEDS/V" H 6150 5300 60  0001 C CNN "Manu-PN"
+F 8 "Wolfson Microelectronics" H 6350 5200 60  0001 C CNN "Manu"
+	1    5800 3950
+	1    0    0    -1
+$EndComp
