File: projects/DAC_L.sch (KiCad schematic (older format))
At the start: 15 parts, among them U401 WM874XX

Commit message: add box cap and small electrolytic cap footprints
Parts:
- removed C402, C404, C406, C408, C410, C412: 22, symbol C
- added C402, C404, C406, C408, C410, C412: 22, symbol CP1
Changed lines of the file:
@@
-$EndComp
-$Comp
-L C C402
-U 1 1 541C1175
-P 3350 4650
-F 0 "C402" H 3350 4750 40  0000 L CNN
-F 1 "22" H 3356 4565 40  0000 L CNN
-F 2 "" H 3388 4500 30  0000 C CNN
-F 3 "" H 3350 4650 60  0000 C CNN
-F 4 "Digi-Key" H 3350 4650 60  0001 C CNN "Supplier"
-F 5 "P16405CT-ND" H 3350 4650 60  0001 C CNN "Supplier-PN"
-F 6 "Panasonic" H 3350 4650 60  0001 C CNN "Manu"
-F 7 "32SEPF22M+TSS" H 3350 4650 60  0001 C CNN "Manu-PN"
-F 8 "CAP ALUM 22UF 32V 20% RADIAL" H 3350 4650 60  0001 C CNN "Description"
-	1    3350 4650
-	1    0    0    -1
 $EndComp
 $Comp
@@
 Connection ~ 7300 2650
 Connection ~ 7300 4450
-$Comp
-L C C404
-U 1 1 544B8579
-P 3850 4650
-F 0 "C404" H 3850 4750 40  0000 L CNN
-F 1 "22" H 3856 4565 40  0000 L CNN
-F 2 "" H 3888 4500 30  0000 C CNN
-F 3 "" H 3850 4650 60  0000 C CNN
-F 4 "Digi-Key" H 3850 4650 60  0001 C CNN "Supplier"
-F 5 "P16405CT-ND" H 3850 4650 60  0001 C CNN "Supplier-PN"
-F 6 "Panasonic" H 3850 4650 60  0001 C CNN "Manu"
-F 7 "32SEPF22M+TSS" H 3850 4650 60  0001 C CNN "Manu-PN"
-F 8 "CAP ALUM 22UF 32V 20% RADIAL" H 3850 4650 60  0001 C CNN "Description"
-	1    3850 4650
-	1    0    0    -1
-$EndComp
-$Comp
-L C C406
-U 1 1 544B857A
-P 4350 4650
-F 0 "C406" H 4350 4750 40  0000 L CNN
-F 1 "22" H 4356 4565 40  0000 L CNN
-F 2 "" H 4388 4500 30  0000 C CNN
-F 3 "" H 4350 4650 60  0000 C CNN
-F 4 "Digi-Key" H 4350 4650 60  0001 C CNN "Supplier"
-F 5 "P16405CT-ND" H 4350 4650 60  0001 C CNN "Supplier-PN"
-F 6 "Panasonic" H 4350 4650 60  0001 C CNN "Manu"
-F 7 "32SEPF22M+TSS" H 4350 4650 60  0001 C CNN "Manu-PN"
-F 8 "CAP ALUM 22UF 32V 20% RADIAL" H 4350 4650 60  0001 C CNN "Description"
-	1    4350 4650
-	1    0    0    -1
-$EndComp
-$Comp
-L C C408
-U 1 1 544B857B
-P 7800 4650
-F 0 "C408" H 7800 4750 40  0000 L CNN
-F 1 "22" H 7806 4565 40  0000 L CNN
-F 2 "" H 7838 4500 30  0000 C CNN
-F 3 "" H 7800 4650 60  0000 C CNN
-F 4 "Digi-Key" H 7800 4650 60  0001 C CNN "Supplier"
-F 5 "P16405CT-ND" H 7800 4650 60  0001 C CNN "Supplier-PN"
-F 6 "Panasonic" H 7800 4650 60  0001 C CNN "Manu"
-F 7 "32SEPF22M+TSS" H 7800 4650 60  0001 C CNN "Manu-PN"
-F 8 "CAP ALUM 22UF 32V 20% RADIAL" H 7800 4650 60  0001 C CNN "Description"
-	1    7800 4650
-	1    0    0    -1
-$EndComp
-$Comp
-L C C410
-U 1 1 544B857C
-P 8300 4650
-F 0 "C410" H 8300 4750 40  0000 L CNN
-F 1 "22" H 8306 4565 40  0000 L CNN
-F 2 "" H 8338 4500 30  0000 C CNN
-F 3 "" H 8300 4650 60  0000 C CNN
-F 4 "Digi-Key" H 8300 4650 60  0001 C CNN "Supplier"
-F 5 "P16405CT-ND" H 8300 4650 60  0001 C CNN "Supplier-PN"
-F 6 "Panasonic" H 8300 4650 60  0001 C CNN "Manu"
-F 7 "32SEPF22M+TSS" H 8300 4650 60  0001 C CNN "Manu-PN"
-F 8 "CAP ALUM 22UF 32V 20% RADIAL" H 8300 4650 60  0001 C CNN "Description"
-	1    8300 4650
-	1    0    0    -1
-$EndComp
-$Comp
-L C C412
-U 1 1 544B857D
-P 8800 4650
-F 0 "C412" H 8800 4750 40  0000 L CNN
-F 1 "22" H 8806 4565 40  0000 L CNN
-F 2 "" H 8838 4500 30  0000 C CNN
-F 3 "" H 8800 4650 60  0000 C CNN
-F 4 "Digi-Key" H 8800 4650 60  0001 C CNN "Supplier"
-F 5 "P16405CT-ND" H 8800 4650 60  0001 C CNN "Supplier-PN"
-F 6 "Panasonic" H 8800 4650 60  0001 C CNN "Manu"
-F 7 "32SEPF22M+TSS" H 8800 4650 60  0001 C CNN "Manu-PN"
-F 8 "CAP ALUM 22UF 32V 20% RADIAL" H 8800 4650 60  0001 C CNN "Description"
-	1    8800 4650
-	1    0    0    -1
-$EndComp
 Wire Wire Line
 	4900 3800 5100 3800
@@
 	9050 4000 9050 5100
 Connection ~ 8800 5100
+$Comp
+L CP1 C402
+U 1 1 54857C2B
+P 3350 4650
+F 0 "C402" H 3400 4750 50  0000 L CNN
+F 1 "22" H 3400 4550 50  0000 L CNN
+F 2 "" H 3350 4650 60  0000 C CNN
+F 3 "" H 3350 4650 60  0000 C CNN
+F 4 "Digi-key" H 3350 4650 60  0001 C CNN "Supplier"
+F 5 "P16405CT-ND" H 3350 4650 60  0001 C CNN "Supplier-PN"
+F 6 "Panasonic" H 3350 4650 60  0001 C CNN "Manu"
+F 7 "32SEPF22M+TSS" H 3350 4650 60  0001 C CNN "Manu-PN"
+F 8 "CAP ALUM 22UF 32V 20% RADIAL" H 3350 4650 60  0001 C CNN "Description"
+	1    3350 4650
+	1    0    0    -1
+$EndComp
+$Comp
+L CP1 C404
+U 1 1 54857D44
+P 3850 4650
+F 0 "C404" H 3900 4750 50  0000 L CNN
+F 1 "22" H 3900 4550 50  0000 L CNN
+F 2 "" H 3850 4650 60  0000 C CNN
+F 3 "" H 3850 4650 60  0000 C CNN
+F 4 "Digi-key" H 3850 4650 60  0001 C CNN "Supplier"
+F 5 "P16405CT-ND" H 3850 4650 60  0001 C CNN "Supplier-PN"
+F 6 "Panasonic" H 3850 4650 60  0001 C CNN "Manu"
+F 7 "32SEPF22M+TSS" H 3850 4650 60  0001 C CNN "Manu-PN"
+F 8 "CAP ALUM 22UF 32V 20% RADIAL" H 3850 4650 60  0001 C CNN "Description"
+	1    3850 4650
+	1    0    0    -1
+$EndComp
+$Comp
+L CP1 C406
+U 1 1 54857D59
+P 4350 4650
+F 0 "C406" H 4400 4750 50  0000 L CNN
+F 1 "22" H 4400 4550 50  0000 L CNN
+F 2 "" H 4350 4650 60  0000 C CNN
+F 3 "" H 4350 4650 60  0000 C CNN
+F 4 "Digi-key" H 4350 4650 60  0001 C CNN "Supplier"
+F 5 "P16405CT-ND" H 4350 4650 60  0001 C CNN "Supplier-PN"
+F 6 "Panasonic" H 4350 4650 60  0001 C CNN "Manu"
+F 7 "32SEPF22M+TSS" H 4350 4650 60  0001 C CNN "Manu-PN"
+F 8 "CAP ALUM 22UF 32V 20% RADIAL" H 4350 4650 60  0001 C CNN "Description"
+	1    4350 4650
+	1    0    0    -1
+$EndComp
+$Comp
+L CP1 C408
+U 1 1 54857D6E
+P 7800 4650
+F 0 "C408" H 7850 4750 50  0000 L CNN
+F 1 "22" H 7850 4550 50  0000 L CNN
+F 2 "" H 7800 4650 60  0000 C CNN
+F 3 "" H 7800 4650 60  0000 C CNN
+F 4 "Digi-key" H 7800 4650 60  0001 C CNN "Supplier"
+F 5 "P16405CT-ND" H 7800 4650 60  0001 C CNN "Supplier-PN"
+F 6 "Panasonic" H 7800 4650 60  0001 C CNN "Manu"
+F 7 "32SEPF22M+TSS" H 7800 4650 60  0001 C CNN "Manu-PN"
+F 8 "CAP ALUM 22UF 32V 20% RADIAL" H 7800 4650 60  0001 C CNN "Description"
+	1    7800 4650
+	1    0    0    -1
+$EndComp
+$Comp
+L CP1 C410
+U 1 1 54857D97
+P 8300 4650
+F 0 "C410" H 8350 4750 50  0000 L CNN
+F 1 "22" H 8350 4550 50  0000 L CNN
+F 2 "" H 8300 4650 60  0000 C CNN
+F 3 "" H 8300 4650 60  0000 C CNN
+F 4 "Digi-key" H 8300 4650 60  0001 C CNN "Supplier"
+F 5 "P16405CT-ND" H 8300 4650 60  0001 C CNN "Supplier-PN"
+F 6 "Panasonic" H 8300 4650 60  0001 C CNN "Manu"
+F 7 "32SEPF22M+TSS" H 8300 4650 60  0001 C CNN "Manu-PN"
+F 8 "CAP ALUM 22UF 32V 20% RADIAL" H 8300 4650 60  0001 C CNN "Description"
+	1    8300 4650
+	1    0    0    -1
+$EndComp
+$Comp
+L CP1 C412
+U 1 1 54857DAC
+P 8800 4650
+F 0 "C412" H 8850 4750 50  0000 L CNN
+F 1 "22" H 8850 4550 50  0000 L CNN
+F 2 "" H 8800 4650 60  0000 C CNN
+F 3 "" H 8800 4650 60  0000 C CNN
+F 4 "Digi-key" H 8800 4650 60  0001 C CNN "Supplier"
+F 5 "P16405CT-ND" H 8800 4650 60  0001 C CNN "Supplier-PN"
+F 6 "Panasonic" H 8800 4650 60  0001 C CNN "Manu"
+F 7 "32SEPF22M+TSS" H 8800 4650 60  0001 C CNN "Manu-PN"
+F 8 "CAP ALUM 22UF 32V 20% RADIAL" H 8800 4650 60  0001 C CNN "Description"
+	1    8800 4650
+	1    0    0    -1
+$EndComp
 $EndSCHEMATC

Commit message: update bom
Parts:
- U401: value WM874XX -> WM8741
Changed lines of the file:
@@
 P 5800 3950
 F 0 "U401" H 5800 3950 60  0000 C CNN
-F 1 "WM874XX" H 5850 4750 60  0000 C CNN
+F 1 "WM8741" H 5850 4750 60  0000 C CNN
 F 2 "" H 5800 3750 60  0000 C CNN
 F 3 "" H 5800 3750 60  0000 C CNN

Commit message: re-add netlist, correct part numbers
Parts:
- removed U401: WM8741, symbol WM874XX
- added U401: WM8741, symbol WM8741
Changed lines of the file:
@@
 LIBS:ti_gosselin
 LIBS:oscillator_gosselin
-LIBS:wolfson_gosselin
 LIBS:power
 LIBS:device
@@
 LIBS:linear_technology_gosselin
 LIBS:led_gosselin
-LIBS:mStereo2-cache
+LIBS:wolfson_gosselin
 EELAYER 24 0
 EELAYER END
@@
 Comment4 ""
 $EndDescr
-$Comp
-L WM874XX U401
-U 1 1 541316E3
-P 5800 3950
-F 0 "U401" H 5800 3950 60  0000 C CNN
-F 1 "WM8741" H 5850 4750 60  0000 C CNN
-F 2 "" H 5800 3750 60  0000 C CNN
-F 3 "" H 5800 3750 60  0000 C CNN
-F 4 "Mouser" H 5950 5000 60  0001 C CNN "Supplier"
-F 5 "238-WM8741GEDS/V" H 6300 5100 60  0001 C CNN "Supplier-PN"
-F 6 "Wolfson Microelectronics" H 6350 5200 60  0001 C CNN "Manu"
-F 7 "WM8741GEDS/V" H 6150 5300 60  0001 C CNN "Manu-PN"
-F 8 "Audio D/A Converter ICs Stereo DAC, High End " H 6900 5400 60  0001 C CNN "Description"
-	1    5800 3950
-	1    0    0    -1
-$EndComp
 Text HLabel 4750 3300 0    60   Input ~ 0
 LRCLK
@@
 	1    0    0    -1
 $EndComp
+$Comp
+L WM8741 U401
+U 1 1 54D07979
+P 5800 3950
+F 0 "U401" H 5800 3950 60  0000 C CNN
+F 1 "WM8741" H 5850 4750 60  0000 C CNN
+F 2 "" H 5800 3750 60  0000 C CNN
+F 3 "" H 5800 3750 60  0000 C CNN
+F 4 "238-WM8741GEDS/V" H 6300 5100 60  0001 C CNN "Supplier-PN"
+F 5 "Mouser" H 5950 5000 60  0001 C CNN "Supplier"
+F 6 "Audio D/A Converter ICs Stereo DAC, High End " H 6900 5400 60  0001 C CNN "Description"
+F 7 "WM8741GEDS/V" H 6150 5300 60  0001 C CNN "Manu-PN"
+F 8 "Wolfson Microelectronics" H 6350 5200 60  0001 C CNN "Manu"
+	1    5800 3950
+	1    0    0    -1
+$EndComp
