File: projects/filter.sch (KiCad schematic (older format))
At the start: 24 parts, among them U601 OPA1632, U602 OPA1632

Commit message: re-re-annotate to remove lowercase
Parts:
- renumbered c601 to C601, c602 to C602, c603 to C603, c604 to C604, C601 to C605, C602 to C606, C603 to C607, C604 to C608
Changed lines of the file:
@@
 LIBS:led_gosselin
 LIBS:wolfson_gosselin
+LIBS:mStereo2-cache
 EELAYER 24 0
 EELAYER END
 $Descr A4 11693 8268
 encoding utf-8
-Sheet 7 7
+Sheet 6 7
 Title ""
 Date ""
@@
 GND
 $Comp
-L C C603
+L C C607
 U 1 1 5428A511
 P 5850 3900
-AR Path="/541690F5/5428A511" Ref="C603"  Part="1"
-AR Path="/5428BABE/5428A511" Ref="C703"  Part="1"
-F 0 "C703" H 5850 4000 40  0000 L CNN
+AR Path="/541690F5/5428A511" Ref="C607"  Part="1"
+AR Path="/5428BABE/5428A511" Ref="C707"  Part="1"
+F 0 "C707" H 5850 4000 40  0000 L CNN
 F 1 "470p" H 5856 3815 40  0000 L CNN
 F 2 "" H 5888 3750 30  0000 C CNN
@@
 $EndComp
 $Comp
-L C C604
+L C C608
 U 1 1 5431DDDC
 P 7950 3900
-AR Path="/541690F5/5431DDDC" Ref="C604"  Part="1"
-AR Path="/5428BABE/5431DDDC" Ref="C704"  Part="1"
-F 0 "C704" H 7950 4000 40  0000 L CNN
+AR Path="/541690F5/5431DDDC" Ref="C608"  Part="1"
+AR Path="/5428BABE/5431DDDC" Ref="C708"  Part="1"
+F 0 "C708" H 7950 4000 40  0000 L CNN
 F 1 "470p" H 7956 3815 40  0000 L CNN
 F 2 "" H 7988 3750 30  0000 C CNN
@@
 $EndComp
 $Comp
-L C C601
+L C C605
 U 1 1 543A33EF
 P 3450 3900
-AR Path="/541690F5/543A33EF" Ref="C601"  Part="1"
-AR Path="/5428BABE/543A33EF" Ref="C701"  Part="1"
-F 0 "C701" H 3450 4000 40  0000 L CNN
+AR Path="/541690F5/543A33EF" Ref="C605"  Part="1"
+AR Path="/5428BABE/543A33EF" Ref="C705"  Part="1"
+F 0 "C705" H 3450 4000 40  0000 L CNN
 F 1 "0.1" H 3456 3815 40  0000 L CNN
 F 2 "" H 3488 3750 30  0000 C CNN
@@
 Connection ~ 2450 4400
 $Comp
-L C C602
+L C C606
 U 1 1 5449F9E9
 P 3750 3900
-AR Path="/541690F5/5449F9E9" Ref="C602"  Part="1"
-AR Path="/5428BABE/5449F9E9" Ref="C702"  Part="1"
-F 0 "C702" H 3750 4000 40  0000 L CNN
+AR Path="/541690F5/5449F9E9" Ref="C606"  Part="1"
+AR Path="/5428BABE/5449F9E9" Ref="C706"  Part="1"
+F 0 "C706" H 3750 4000 40  0000 L CNN
 F 1 "0.1" H 3756 3815 40  0000 L CNN
 F 2 "" H 3788 3750 30  0000 C CNN
@@
 $EndComp
 $Comp
-L CP1 c601
+L CP1 C601
 U 1 1 548575CB
 P 2100 3650
-AR Path="/541690F5/548575CB" Ref="c601"  Part="1"
-AR Path="/5428BABE/548575CB" Ref="c701"  Part="1"
-F 0 "c701" H 2150 3750 50  0000 L CNN
+AR Path="/541690F5/548575CB" Ref="C601"  Part="1"
+AR Path="/5428BABE/548575CB" Ref="C701"  Part="1"
+F 0 "C701" H 2150 3750 50  0000 L CNN
 F 1 "100" H 2150 3550 50  0000 L CNN
 F 2 "" H 2100 3650 60  0000 C CNN
@@
 $EndComp
 $Comp
-L CP1 c602
+L CP1 C602
 U 1 1 54857740
 P 2100 4150
-AR Path="/541690F5/54857740" Ref="c602"  Part="1"
-AR Path="/5428BABE/54857740" Ref="c702"  Part="1"
-F 0 "c702" H 2150 4250 50  0000 L CNN
+AR Path="/541690F5/54857740" Ref="C602"  Part="1"
+AR Path="/5428BABE/54857740" Ref="C702"  Part="1"
+F 0 "C702" H 2150 4250 50  0000 L CNN
 F 1 "100" H 2150 4050 50  0000 L CNN
 F 2 "" H 2100 4150 60  0000 C CNN
@@
 $EndComp
 $Comp
-L CP1 c603
+L CP1 C603
 U 1 1 54857755
 P 2450 3650
-AR Path="/541690F5/54857755" Ref="c603"  Part="1"
-AR Path="/5428BABE/54857755" Ref="c703"  Part="1"
-F 0 "c703" H 2500 3750 50  0000 L CNN
+AR Path="/541690F5/54857755" Ref="C603"  Part="1"
+AR Path="/5428BABE/54857755" Ref="C703"  Part="1"
+F 0 "C703" H 2500 3750 50  0000 L CNN
 F 1 "100" H 2500 3550 50  0000 L CNN
 F 2 "" H 2450 3650 60  0000 C CNN
@@
 $EndComp
 $Comp
-L CP1 c604
+L CP1 C604
 U 1 1 5485776A
 P 2450 4150
-AR Path="/541690F5/5485776A" Ref="c604"  Part="1"
-AR Path="/5428BABE/5485776A" Ref="c704"  Part="1"
-F 0 "c704" H 2500 4250 50  0000 L CNN
+AR Path="/541690F5/5485776A" Ref="C604"  Part="1"
+AR Path="/5428BABE/5485776A" Ref="C704"  Part="1"
+F 0 "C704" H 2500 4250 50  0000 L CNN
 F 1 "100" H 2500 4050 50  0000 L CNN
 F 2 "" H 2450 4150 60  0000 C CNN
